Commit message: edit ma_robot pkg

File: ma_robot_description/urdf/assemblies/front_left_wheel_link.urdf.xacro (robot description, xacro)
@@ -3,22 +3,22 @@
   <xacro:macro name="front_left_wheel_link" params="prefix">
     <!-- Links -->
-    <link name="${prefix}Part2_1">
+    <link name="${prefix}front_left_wheel_link">
       <inertial>
-        <origin xyz="-0.129964 -0.020034 0.052271" rpy="0 0 0"/>
-        <mass value="0.967990"/>
-        <inertia ixx="4.354820e-04" ixy="-1.765367e-07" ixz="9.904484e-07"
-                 iyy="4.318266e-04" iyz="1.096024e-06" izz="6.297403e-04"/>
+        <origin xyz="-0.000000 -0.000000 -0.007006" rpy="0 0 0"/>
+        <mass value="0.611603"/>
+        <inertia ixx="5.265770e-04" ixy="-5.777757e-10" ixz="8.274260e-11"
+                 iyy="5.265750e-04" iyz="-6.033033e-11" izz="7.325315e-04"/>
       </inertial>
       <visual>
-        <origin xyz="-0.130000 -0.020000 0.070000" rpy="-1.570796 0.000000 0.000000"/>
+        <origin xyz="-0.012900 -0.018048 -0.001523" rpy="1.570796 0.000000 0.000000"/>
         <geometry>
-          <mesh filename="package://ma_robot_description/meshes/front_left_wheel_link/Part2_1.dae" scale="1 1 1"/>
+          <mesh filename="package://ma_robot_description/meshes/front_left_wheel_link/front_left_wheel_link.dae" scale="1 1 1"/>
         </geometry>
         <material name="Steel"/>
       </visual>
       <collision>
-        <origin xyz="-0.130000 -0.020000 0.070000" rpy="-1.570796 0.000000 0.000000"/>
+        <origin xyz="-0.012900 -0.018048 -0.001523" rpy="1.570796 0.000000 0.000000"/>
         <geometry>
-          <mesh filename="package://ma_robot_description/meshes/front_left_wheel_link/Part2_1_collision.stl" scale="0.01 0.01 0.01"/>
+          <mesh filename="package://ma_robot_description/meshes/front_left_wheel_link/front_left_wheel_link_collision.stl" scale="0.01 0.01 0.01"/>
         </geometry>
       </collision>

File: ma_robot_description/urdf/assemblies/front_right_wheel_link.urdf.xacro (robot description, xacro)
@@ -3,22 +3,22 @@
   <xacro:macro name="front_right_wheel_link" params="prefix">
     <!-- Links -->
-    <link name="${prefix}Part2_1_Mirror">
+    <link name="${prefix}front_right_wheel_link">
       <inertial>
-        <origin xyz="-0.129964 -0.019966 -0.185729" rpy="0 0 0"/>
-        <mass value="0.967990"/>
-        <inertia ixx="4.354820e-04" ixy="1.765368e-07" ixz="9.904484e-07"
-                 iyy="4.318266e-04" iyz="-1.096024e-06" izz="6.297403e-04"/>
+        <origin xyz="0.000000 0.000000 -0.007006" rpy="0 0 0"/>
+        <mass value="0.611603"/>
+        <inertia ixx="5.265770e-04" ixy="-5.777757e-10" ixz="-8.274263e-11"
+                 iyy="5.265750e-04" iyz="6.033033e-11" izz="7.325315e-04"/>
       </inertial>
       <visual>
-        <origin xyz="-0.130000 -0.020000 -0.168000" rpy="-1.570796 0.000000 0.000000"/>
+        <origin xyz="0.012900 0.018048 -0.001523" rpy="1.570796 0.000000 3.141593"/>
         <geometry>
-          <mesh filename="package://ma_robot_description/meshes/front_right_wheel_link/Part2_1_Mirror.dae" scale="1 1 1"/>
+          <mesh filename="package://ma_robot_description/meshes/front_right_wheel_link/front_right_wheel_link.dae" scale="1 1 1"/>
         </geometry>
         <material name="Steel"/>
       </visual>
       <collision>
-        <origin xyz="-0.130000 -0.020000 -0.168000" rpy="-1.570796 0.000000 0.000000"/>
+        <origin xyz="0.012900 0.018048 -0.001523" rpy="1.570796 0.000000 3.141593"/>
         <geometry>
-          <mesh filename="package://ma_robot_description/meshes/front_right_wheel_link/Part2_1_Mirror_collision.stl" scale="0.01 0.01 0.01"/>
+          <mesh filename="package://ma_robot_description/meshes/front_right_wheel_link/front_right_wheel_link_collision.stl" scale="0.01 0.01 0.01"/>
         </geometry>
       </collision>

File: ma_robot_description/urdf/assemblies/ma_robot.urdf.xacro (robot description, xacro)
@@ -5,9 +5,16 @@
     <link name="${prefix}base_link">
       <inertial>
-        <origin xyz="0.041574 -0.062494 0.024420" rpy="0 0 0"/>
-        <mass value="2.899152"/>
-        <inertia ixx="7.973742e-03" ixy="9.036729e-07" ixz="2.781740e-04"
-                 iyy="1.379462e-02" iyz="-4.481306e-07" izz="2.052761e-02"/>
+        <origin xyz="0.041573 -0.062494 0.024421" rpy="0 0 0"/>
+        <mass value="2.899175"/>
+        <inertia ixx="7.973873e-03" ixy="9.036956e-07" ixz="2.783768e-04"
+                 iyy="1.379507e-02" iyz="-4.481468e-07" izz="2.052792e-02"/>
       </inertial>
+      <visual>
+        <origin xyz="0.000000 0.000000 0.000000" rpy="0.000000 0.000000 0.000000"/>
+        <geometry>
+          <mesh filename="package://ma_robot_description/meshes/ma_robot/base_link.dae" scale="1 1 1"/>
+        </geometry>
+        <material name="Acetal_Resin_Black"/>
+      </visual>
       <collision>
         <origin xyz="0.000000 0.000000 0.000000" rpy="0.000000 0.000000 0.000000"/>
@@ -17,57 +24,4 @@
       </collision>
     </link>
-    <link name="${prefix}zed2_camera_link">
-      <inertial>
-        <origin xyz="0.000000 0.015505 0.042389" rpy="0 0 0"/>
-        <mass value="0.178229"/>
-        <inertia ixx="2.662726e-05" ixy="-3.215230e-09" ixz="-1.621734e-09"
-                 iyy="4.362977e-04" iyz="-2.967393e-09" izz="4.390806e-04"/>
-      </inertial>
-      <visual>
-        <origin xyz="0.000000 0.000000 0.000000" rpy="0.000000 0.000000 0.000000"/>
-        <geometry>
-          <mesh filename="package://ma_robot_description/meshes/ma_robot/zed2_camera_link.dae" scale="1 1 1"/>
-        </geometry>
-        <material name="PA_11_Nylon_HP_11_30_with_EOS_P_396_3D_Printer"/>
-      </visual>
-      <collision>
-        <origin xyz="0.000000 0.000000 0.000000" rpy="0.000000 0.000000 0.000000"/>
-        <geometry>
-          <mesh filename="package://ma_robot_description/meshes/ma_robot/zed2_camera_link_collision.stl" scale="0.01 0.01 0.01"/>
-        </geometry>
-      </collision>
-    </link>
-    <link name="${prefix}rplidar_s2_link">
-      <inertial>
-        <origin xyz="-0.595013 0.532942 0.012880" rpy="0 0 0"/>
-        <mass value="0.203764"/>
-        <inertia ixx="1.351079e-04" ixy="-7.653496e-09" ixz="1.410544e-08"
-                 iyy="1.362177e-04" iyz="3.930765e-08" izz="2.370283e-04"/>
-      </inertial>
-      <visual>
-        <origin xyz="0.000000 0.000000 0.000000" rpy="0.000000 0.000000 0.000000"/>
-        <geometry>
-          <mesh filename="package://ma_robot_description/meshes/ma_robot/rplidar_s2_link.dae" scale="1 1 1"/>
-        </geometry>
-        <material name="Steel"/>
-      </visual>
-      <collision>
-        <origin xyz="0.000000 0.000000 0.000000" rpy="0.000000 0.000000 0.000000"/>
-        <geometry>
-          <mesh filename="package://ma_robot_description/meshes/ma_robot/rplidar_s2_link_collision.stl" scale="0.01 0.01 0.01"/>
-        </geometry>
-      </collision>
-    </link>
-    <!-- Joints (internal to assembly) -->
-    <joint name="${prefix}Rigid_1" type="fixed">
-      <parent link="${prefix}base_link"/>
-      <child link="${prefix}zed2_camera_link"/>
-      <origin xyz="0.145000 -0.062500 -0.007371" rpy="0.000000 0.000000 -1.570796"/>
-    </joint>
-    <joint name="${prefix}Rigid_2" type="fixed">
-      <parent link="${prefix}base_link"/>
-      <child link="${prefix}rplidar_s2_link"/>
-      <origin xyz="-0.433747 -0.657506 0.046815" rpy="0.000000 0.000000 -1.570796"/>
-    </joint>
   </xacro:macro>
 </robot>

File: ma_robot_description/urdf/assemblies/rear_left_wheel_link.urdf.xacro (robot description, xacro)
@@ -3,22 +3,22 @@
   <xacro:macro name="rear_left_wheel_link" params="prefix">
     <!-- Links -->
-    <link name="${prefix}Part2_2_Mirror">
+    <link name="${prefix}rear_left_wheel_link">
       <inertial>
-        <origin xyz="0.020036 -0.019966 0.025271" rpy="0 0 0"/>
-        <mass value="0.967990"/>
-        <inertia ixx="4.354820e-04" ixy="1.765368e-07" ixz="9.904484e-07"
-                 iyy="4.318266e-04" iyz="-1.096024e-06" izz="6.297403e-04"/>
+        <origin xyz="-0.000000 -0.000000 -0.007006" rpy="0 0 0"/>
+        <mass value="0.611603"/>
+        <inertia ixx="5.265770e-04" ixy="-5.777757e-10" ixz="8.274260e-11"
+                 iyy="5.265750e-04" iyz="-6.033033e-11" izz="7.325315e-04"/>
       </inertial>
       <visual>
-        <origin xyz="0.020000 -0.020000 0.043000" rpy="-1.570796 0.000000 0.000000"/>
+        <origin xyz="-0.012900 -0.018048 -0.001523" rpy="1.570796 0.000000 0.000000"/>
         <geometry>
-          <mesh filename="package://ma_robot_description/meshes/rear_left_wheel_link/Part2_2_Mirror.dae" scale="1 1 1"/>
+          <mesh filename="package://ma_robot_description/meshes/rear_left_wheel_link/rear_left_wheel_link.dae" scale="1 1 1"/>
         </geometry>
         <material name="Steel"/>
       </visual>
       <collision>
-        <origin xyz="0.020000 -0.020000 0.043000" rpy="-1.570796 0.000000 0.000000"/>
+        <origin xyz="-0.012900 -0.018048 -0.001523" rpy="1.570796 0.000000 0.000000"/>
         <geometry>
-          <mesh filename="package://ma_robot_description/meshes/rear_left_wheel_link/Part2_2_Mirror_collision.stl" scale="0.01 0.01 0.01"/>
+          <mesh filename="package://ma_robot_description/meshes/rear_left_wheel_link/rear_left_wheel_link_collision.stl" scale="0.01 0.01 0.01"/>
         </geometry>
       </collision>

File: ma_robot_description/urdf/assemblies/rear_right_wheel_link.urdf.xacro (robot description, xacro)
@@ -3,22 +3,22 @@
   <xacro:macro name="rear_right_wheel_link" params="prefix">
     <!-- Links -->
-    <link name="${prefix}Part2_2">
+    <link name="${prefix}rear_right_wheel_link">
       <inertial>
-        <origin xyz="0.020036 -0.020034 -0.185729" rpy="0 0 0"/>
-        <mass value="0.967990"/>
-        <inertia ixx="4.354820e-04" ixy="-1.765367e-07" ixz="9.904484e-07"
-                 iyy="4.318266e-04" iyz="1.096024e-06" izz="6.297403e-04"/>
+        <origin xyz="0.000000 0.000000 -0.009006" rpy="0 0 0"/>
+        <mass value="0.611603"/>
+        <inertia ixx="5.265770e-04" ixy="-5.777757e-10" ixz="-8.274261e-11"
+                 iyy="5.265750e-04" iyz="6.033033e-11" izz="7.325315e-04"/>
       </inertial>
       <visual>
-        <origin xyz="0.020000 -0.020000 -0.168000" rpy="-1.570796 0.000000 0.000000"/>
+        <origin xyz="0.012900 0.018048 -0.003523" rpy="1.570796 0.000000 3.141593"/>
         <geometry>
-          <mesh filename="package://ma_robot_description/meshes/rear_right_wheel_link/Part2_2.dae" scale="1 1 1"/>
+          <mesh filename="package://ma_robot_description/meshes/rear_right_wheel_link/rear_right_wheel_link.dae" scale="1 1 1"/>
         </geometry>
         <material name="Steel"/>
       </visual>
       <collision>
-        <origin xyz="0.020000 -0.020000 -0.168000" rpy="-1.570796 0.000000 0.000000"/>
+        <origin xyz="0.012900 0.018048 -0.003523" rpy="1.570796 0.000000 3.141593"/>
         <geometry>
-          <mesh filename="package://ma_robot_description/meshes/rear_right_wheel_link/Part2_2_collision.stl" scale="0.01 0.01 0.01"/>
+          <mesh filename="package://ma_robot_description/meshes/rear_right_wheel_link/rear_right_wheel_link_collision.stl" scale="0.01 0.01 0.01"/>
         </geometry>
       </collision>

File: ma_robot_description/urdf/ma_robot.urdf (robot description, URDF)
Before this commit: robot ma_robot, 7 links, 6 joints
Links:
- removed link Part2_1
- removed link Part2_1_Mirror
- removed link Part2_2
- removed link Part2_2_Mirror
- added link front_left_wheel_link, mass 0.611603; collision mesh filename=package://ma_robot_description/meshes/front_left_wheel_link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 scale=0.01 0.01 0.01; visual mesh filename=package://ma_robot_description/meshes/front_left_wheel_link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 scale=1 1 1
- added link front_right_wheel_link, mass 0.611603; collision mesh filename=package://ma_robot_description/meshes/front_right_wheel_lin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 scale=0.01 0.01 0.01; visual mesh filename=package://ma_robot_description/meshes/front_right_wheel_lin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 scale=1 1 1
- added link rear_left_wheel_link, mass 0.611603; collision mesh filename=package://ma_robot_description/meshes/rear_left_wheel_link/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 scale=0.01 0.01 0.01; visual mesh filename=package://ma_robot_description/meshes/rear_left_wheel_link/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 scale=1 1 1
- added link rear_right_wheel_link, mass 0.611603; collision mesh filename=package://ma_robot_description/meshes/rear_right_wheel_link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 scale=0.01 0.01 0.01; visual mesh filename=package://ma_robot_description/meshes/rear_right_wheel_link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 scale=1 1 1
- link base_link: mass 2.899152 -> 2.899175; geometry collision mesh filename=package://ma_robot_description/meshes/ma_robot/base_link_co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 scale=0.01 0.01 0.01; visual mesh filename=package://ma_robot_description/meshes/ma_robot/base_link.dae scale=1 1 1
- link rplidar_s2_link: geometry collision mesh filename=package://ma_robot_description/meshes/base_link/rplidar_s2_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 scale=0.01 0.01 0.01; visual mesh filename=package://ma_robot_description/meshes/base_link/rplidar_s2_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 scale=1 1 1
- link zed2_camera_link: geometry collision mesh filename=package://ma_robot_description/meshes/base_link/zed2_camera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 scale=0.01 0.01 0.01; visual mesh filename=package://ma_robot_description/meshes/base_link/zed2_camera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 scale=1 1 1
Joints:
- removed joint Revolute_5
- removed joint Revolute_6
- removed joint Revolute_8
- removed joint Revolute_9
- removed joint Rigid_1
- removed joint Rigid_2
- added joint front_left_wheel_joint: type continuous, parent base_link, child front_left_wheel_link, origin xyz=0.130000 0.060000 0.020000 rpy=-1.570796 0.000000 0.000000, axis 0.000000 0.000000 1.000000, limit effort=100.0 velocity=1.00
- added joint front_right_wheel_joint: type continuous, parent base_link, child front_right_wheel_link, origin xyz=0.130000 -0.185000 0.020000 rpy=1.570796 0.000000 0.000000, axis 0.000000 0.000000 1.000000, limit effort=100.0 velocity=1.00
- added joint rear_left_wheel_joint: type continuous, parent base_link, child rear_left_wheel_link, origin xyz=-0.020000 0.060000 0.020000 rpy=-1.570796 0.000000 0.000000, axis 0.000000 0.000000 1.000000, limit effort=100.0 velocity=1.00
- added joint rear_right_wheel_joint: type continuous, parent base_link, child rear_right_wheel_link, origin xyz=-0.020000 -0.187000 0.020000 rpy=1.570796 0.000000 0.000000, axis 0.000000 0.000000 1.000000, limit effort=100.0 velocity=1.00
- added joint rplidar_s2_joint: type fixed, parent base_link, child rplidar_s2_link, origin xyz=-0.433747 -0.657506 0.046815 rpy=0.000000 0.000000 -1.570796
- added joint zed2_camera_joint: type fixed, parent base_link, child zed2_camera_link, origin xyz=0.145000 -0.062500 -0.007371 rpy=0.000000 0.000000 -1.570796

File: ma_robot_description/urdf/ma_robot.urdf.xacro (robot description, xacro)
@@ -13,13 +13,15 @@
   <!-- Assembly includes -->
   <xacro:include filename="$(find ma_robot_description)/urdf/assemblies/front_left_wheel_link.urdf.xacro"/>
-  <xacro:include filename="$(find ma_robot_description)/urdf/assemblies/rear_right_wheel_link.urdf.xacro"/>
   <xacro:include filename="$(find ma_robot_description)/urdf/assemblies/front_right_wheel_link.urdf.xacro"/>
   <xacro:include filename="$(find ma_robot_description)/urdf/assemblies/rear_left_wheel_link.urdf.xacro"/>
+  <xacro:include filename="$(find ma_robot_description)/urdf/assemblies/rear_right_wheel_link.urdf.xacro"/>
+  <xacro:include filename="$(find ma_robot_description)/urdf/assemblies/base_link.urdf.xacro"/>
   <xacro:include filename="$(find ma_robot_description)/urdf/assemblies/ma_robot.urdf.xacro"/>
   <!-- Instantiate assemblies -->
   <xacro:front_left_wheel_link prefix=""/>
-  <xacro:rear_right_wheel_link prefix=""/>
   <xacro:front_right_wheel_link prefix=""/>
   <xacro:rear_left_wheel_link prefix=""/>
+  <xacro:rear_right_wheel_link prefix=""/>
+  <xacro:base_link prefix=""/>
   <xacro:ma_robot prefix=""/>
   <!-- Mount joints (cross-assembly connections) -->
@@ -28,29 +30,39 @@
   <!-- update the include + macro call above, and adjust -->
   <!-- parent/child link names in the mount joint below. -->
-  <joint name="Revolute_5" type="continuous">
+  <joint name="zed2_camera_joint" type="fixed">
     <parent link="base_link"/>
-    <child link="Part2_1"/>
-    <origin xyz="0.260000 0.000000 0.000000" rpy="-1.570796 0.000000 0.000000"/>
+    <child link="zed2_camera_link"/>
+    <origin xyz="0.145000 -0.062500 -0.007371" rpy="0.000000 0.000000 -1.570796"/>
+  </joint>
+  <joint name="rplidar_s2_joint" type="fixed">
+    <parent link="base_link"/>
+    <child link="rplidar_s2_link"/>
+    <origin xyz="-0.433747 -0.657506 0.046815" rpy="0.000000 0.000000 -1.570796"/>
+  </joint>
+  <joint name="front_right_wheel_joint" type="continuous">
+    <parent link="base_link"/>
+    <child link="front_right_wheel_link"/>
+    <origin xyz="0.130000 -0.185000 0.020000" rpy="1.570796 0.000000 0.000000"/>
     <axis xyz="0.000000 0.000000 1.000000"/>
     <limit effort="100.0" velocity="1.00"/>
   </joint>
-  <joint name="Revolute_6" type="continuous">
+  <joint name="rear_right_wheel_joint" type="continuous">
     <parent link="base_link"/>
-    <child link="Part2_2"/>
-    <origin xyz="-0.040000 -0.362000 0.040000" rpy="1.570796 0.000000 0.000000"/>
+    <child link="rear_right_wheel_link"/>
+    <origin xyz="-0.020000 -0.187000 0.020000" rpy="1.570796 0.000000 0.000000"/>
     <axis xyz="0.000000 0.000000 1.000000"/>
     <limit effort="100.0" velocity="1.00"/>
   </joint>
-  <joint name="Revolute_8" type="continuous">
+  <joint name="front_left_wheel_joint" type="continuous">
     <parent link="base_link"/>
-    <child link="Part2_1_Mirror"/>
-    <origin xyz="0.260000 -0.362000 0.040000" rpy="1.570796 0.000000 0.000000"/>
+    <child link="front_left_wheel_link"/>
+    <origin xyz="0.130000 0.060000 0.020000" rpy="-1.570796 0.000000 0.000000"/>
     <axis xyz="0.000000 0.000000 1.000000"/>
     <limit effort="100.0" velocity="1.00"/>
   </joint>
-  <joint name="Revolute_9" type="continuous">
+  <joint name="rear_left_wheel_joint" type="continuous">
     <parent link="base_link"/>
-    <child link="Part2_2_Mirror"/>
-    <origin xyz="-0.040000 0.026000 0.000000" rpy="-1.570796 0.000000 0.000000"/>
+    <child link="rear_left_wheel_link"/>
+    <origin xyz="-0.020000 0.060000 0.020000" rpy="-1.570796 0.000000 0.000000"/>
     <axis xyz="0.000000 0.000000 1.000000"/>
     <limit effort="100.0" velocity="1.00"/>
@@ -63,5 +75,5 @@
       <param name="state_topic">sim/ma_robot_system/state</param>
     </hardware>
-    <joint name="Revolute_5">
+    <joint name="front_left_wheel_joint">
       <command_interface name="position"/>
       <command_interface name="velocity"/>
@@ -72,5 +84,5 @@
       <state_interface name="effort"/>
     </joint>
-    <joint name="Revolute_6">
+    <joint name="front_right_wheel_joint">
       <command_interface name="position"/>
       <command_interface name="velocity"/>
@@ -81,5 +93,5 @@
       <state_interface name="effort"/>
     </joint>
-    <joint name="Revolute_8">
+    <joint name="rear_left_wheel_joint">
       <command_interface name="position"/>
       <command_interface name="velocity"/>
@@ -90,5 +102,5 @@
       <state_interface name="effort"/>
     </joint>
-    <joint name="Revolute_9">
+    <joint name="rear_right_wheel_joint">
       <command_interface name="position"/>
       <command_interface name="velocity"/>
