Commit message: edit ma_robot pkg

File: ma_robot_description/urdf/assemblies/front_left_wheel_link.urdf.xacro (robot description, xacro)
@@ -5,11 +5,11 @@
     <link name="${prefix}front_left_wheel_link">
       <inertial>
-        <origin xyz="-0.000000 -0.000000 -0.007006" rpy="0 0 0"/>
+        <origin xyz="0.117100 -0.063048 -0.068483" rpy="0 0 0"/>
         <mass value="0.611603"/>
-        <inertia ixx="5.265770e-04" ixy="-5.777757e-10" ixz="8.274260e-11"
-                 iyy="5.265750e-04" iyz="-6.033033e-11" izz="7.325315e-04"/>
+        <inertia ixx="5.265770e-04" ixy="-5.777757e-10" ixz="-8.274260e-11"
+                 iyy="5.265750e-04" iyz="6.033033e-11" izz="7.325315e-04"/>
       </inertial>
       <visual>
-        <origin xyz="-0.012900 -0.018048 -0.001523" rpy="1.570796 0.000000 0.000000"/>
+        <origin xyz="0.130000 -0.045000 -0.063000" rpy="1.570796 0.000000 3.141593"/>
         <geometry>
           <mesh filename="package://ma_robot_description/meshes/front_left_wheel_link/front_left_wheel_link.dae" scale="1 1 1"/>
@@ -18,5 +18,5 @@
       </visual>
       <collision>
-        <origin xyz="-0.012900 -0.018048 -0.001523" rpy="1.570796 0.000000 0.000000"/>
+        <origin xyz="0.130000 -0.045000 -0.063000" rpy="1.570796 0.000000 3.141593"/>
         <geometry>
           <mesh filename="package://ma_robot_description/meshes/front_left_wheel_link/front_left_wheel_link_collision.stl" scale="0.01 0.01 0.01"/>

File: ma_robot_description/urdf/assemblies/front_right_wheel_link.urdf.xacro (robot description, xacro)
@@ -5,11 +5,11 @@
     <link name="${prefix}front_right_wheel_link">
       <inertial>
-        <origin xyz="0.000000 0.000000 -0.007006" rpy="0 0 0"/>
+        <origin xyz="0.117100 -0.063048 0.183517" rpy="0 0 0"/>
         <mass value="0.611603"/>
-        <inertia ixx="5.265770e-04" ixy="-5.777757e-10" ixz="-8.274263e-11"
+        <inertia ixx="5.265770e-04" ixy="-5.777757e-10" ixz="-8.274258e-11"
                  iyy="5.265750e-04" iyz="6.033033e-11" izz="7.325315e-04"/>
       </inertial>
       <visual>
-        <origin xyz="0.012900 0.018048 -0.001523" rpy="1.570796 0.000000 3.141593"/>
+        <origin xyz="0.130000 -0.045000 0.189000" rpy="1.570796 0.000000 3.141593"/>
         <geometry>
           <mesh filename="package://ma_robot_description/meshes/front_right_wheel_link/front_right_wheel_link.dae" scale="1 1 1"/>
@@ -18,5 +18,5 @@
       </visual>
       <collision>
-        <origin xyz="0.012900 0.018048 -0.001523" rpy="1.570796 0.000000 3.141593"/>
+        <origin xyz="0.130000 -0.045000 0.189000" rpy="1.570796 0.000000 3.141593"/>
         <geometry>
           <mesh filename="package://ma_robot_description/meshes/front_right_wheel_link/front_right_wheel_link_collision.stl" scale="0.01 0.01 0.01"/>

File: ma_robot_description/urdf/assemblies/ma_robot.urdf.xacro (robot description, xacro)
@@ -5,8 +5,8 @@
     <link name="${prefix}base_link">
       <inertial>
-        <origin xyz="0.041573 -0.062494 0.024421" rpy="0 0 0"/>
-        <mass value="2.899175"/>
-        <inertia ixx="7.973873e-03" ixy="9.036956e-07" ixz="2.783768e-04"
-                 iyy="1.379507e-02" iyz="-4.481468e-07" izz="2.052792e-02"/>
+        <origin xyz="0.041574 -0.062494 0.024420" rpy="0 0 0"/>
+        <mass value="2.899172"/>
+        <inertia ixx="7.973854e-03" ixy="9.036948e-07" ixz="2.783510e-04"
+                 iyy="1.379501e-02" iyz="-4.481462e-07" izz="2.052789e-02"/>
       </inertial>
       <visual>
@@ -24,4 +24,57 @@
       </collision>
     </link>
+    <link name="${prefix}zed2_camera_link">
+      <inertial>
+        <origin xyz="0.000000 0.015505 0.042389" rpy="0 0 0"/>
+        <mass value="0.178229"/>
+        <inertia ixx="2.662726e-05" ixy="-3.215230e-09" ixz="-1.621734e-09"
+                 iyy="4.362977e-04" iyz="-2.967393e-09" izz="4.390806e-04"/>
+      </inertial>
+      <visual>
+        <origin xyz="0.000000 0.000000 0.000000" rpy="0.000000 0.000000 0.000000"/>
+        <geometry>
+          <mesh filename="package://ma_robot_description/meshes/ma_robot/zed2_camera_link.dae" scale="1 1 1"/>
+        </geometry>
+        <material name="PA_11_Nylon_HP_11_30_with_EOS_P_396_3D_Printer"/>
+      </visual>
+      <collision>
+        <origin xyz="0.000000 0.000000 0.000000" rpy="0.000000 0.000000 0.000000"/>
+        <geometry>
+          <mesh filename="package://ma_robot_description/meshes/ma_robot/zed2_camera_link_collision.stl" scale="0.01 0.01 0.01"/>
+        </geometry>
+      </collision>
+    </link>
+    <link name="${prefix}rplidar_s2_link">
+      <inertial>
+        <origin xyz="-0.595013 0.532942 0.012880" rpy="0 0 0"/>
+        <mass value="0.203764"/>
+        <inertia ixx="1.351079e-04" ixy="-7.653496e-09" ixz="1.410544e-08"
+                 iyy="1.362177e-04" iyz="3.930765e-08" izz="2.370283e-04"/>
+      </inertial>
+      <visual>
+        <origin xyz="0.000000 0.000000 0.000000" rpy="0.000000 0.000000 0.000000"/>
+        <geometry>
+          <mesh filename="package://ma_robot_description/meshes/ma_robot/rplidar_s2_link.dae" scale="1 1 1"/>
+        </geometry>
+        <material name="Steel"/>
+      </visual>
+      <collision>
+        <origin xyz="0.000000 0.000000 0.000000" rpy="0.000000 0.000000 0.000000"/>
+        <geometry>
+          <mesh filename="package://ma_robot_description/meshes/ma_robot/rplidar_s2_link_collision.stl" scale="0.01 0.01 0.01"/>
+        </geometry>
+      </collision>
+    </link>
+    <!-- Joints (internal to assembly) -->
+    <joint name="${prefix}zed2_camera_joint" type="fixed">
+      <parent link="${prefix}base_link"/>
+      <child link="${prefix}zed2_camera_link"/>
+      <origin xyz="0.145000 -0.062500 -0.007371" rpy="0.000000 0.000000 -1.570796"/>
+    </joint>
+    <joint name="${prefix}rplidar_s2_joint" type="fixed">
+      <parent link="${prefix}base_link"/>
+      <child link="${prefix}rplidar_s2_link"/>
+      <origin xyz="-0.433747 -0.657506 0.046815" rpy="0.000000 0.000000 -1.570796"/>
+    </joint>
   </xacro:macro>
 </robot>

File: ma_robot_description/urdf/assemblies/rear_left_wheel_link.urdf.xacro (robot description, xacro)
@@ -5,5 +5,5 @@
     <link name="${prefix}rear_left_wheel_link">
       <inertial>
-        <origin xyz="-0.000000 -0.000000 -0.007006" rpy="0 0 0"/>
+        <origin xyz="0.032900 0.063048 -0.075483" rpy="0 0 0"/>
         <mass value="0.611603"/>
         <inertia ixx="5.265770e-04" ixy="-5.777757e-10" ixz="8.274260e-11"
@@ -11,5 +11,5 @@
       </inertial>
       <visual>
-        <origin xyz="-0.012900 -0.018048 -0.001523" rpy="1.570796 0.000000 0.000000"/>
+        <origin xyz="0.020000 0.045000 -0.070000" rpy="1.570796 0.000000 0.000000"/>
         <geometry>
           <mesh filename="package://ma_robot_description/meshes/rear_left_wheel_link/rear_left_wheel_link.dae" scale="1 1 1"/>
@@ -18,5 +18,5 @@
       </visual>
       <collision>
-        <origin xyz="-0.012900 -0.018048 -0.001523" rpy="1.570796 0.000000 0.000000"/>
+        <origin xyz="0.020000 0.045000 -0.070000" rpy="1.570796 0.000000 0.000000"/>
         <geometry>
           <mesh filename="package://ma_robot_description/meshes/rear_left_wheel_link/rear_left_wheel_link_collision.stl" scale="0.01 0.01 0.01"/>

File: ma_robot_description/urdf/assemblies/rear_right_wheel_link.urdf.xacro (robot description, xacro)
@@ -5,11 +5,11 @@
     <link name="${prefix}rear_right_wheel_link">
       <inertial>
-        <origin xyz="0.000000 0.000000 -0.009006" rpy="0 0 0"/>
+        <origin xyz="0.032900 0.063048 0.183517" rpy="0 0 0"/>
         <mass value="0.611603"/>
-        <inertia ixx="5.265770e-04" ixy="-5.777757e-10" ixz="-8.274261e-11"
-                 iyy="5.265750e-04" iyz="6.033033e-11" izz="7.325315e-04"/>
+        <inertia ixx="5.265770e-04" ixy="-5.777757e-10" ixz="8.274260e-11"
+                 iyy="5.265750e-04" iyz="-6.033033e-11" izz="7.325315e-04"/>
       </inertial>
       <visual>
-        <origin xyz="0.012900 0.018048 -0.003523" rpy="1.570796 0.000000 3.141593"/>
+        <origin xyz="0.020000 0.045000 0.189000" rpy="1.570796 0.000000 0.000000"/>
         <geometry>
           <mesh filename="package://ma_robot_description/meshes/rear_right_wheel_link/rear_right_wheel_link.dae" scale="1 1 1"/>
@@ -18,5 +18,5 @@
       </visual>
       <collision>
-        <origin xyz="0.012900 0.018048 -0.003523" rpy="1.570796 0.000000 3.141593"/>
+        <origin xyz="0.020000 0.045000 0.189000" rpy="1.570796 0.000000 0.000000"/>
         <geometry>
           <mesh filename="package://ma_robot_description/meshes/rear_right_wheel_link/rear_right_wheel_link_collision.stl" scale="0.01 0.01 0.01"/>

File: ma_robot_description/urdf/ma_robot.urdf (robot description, URDF)
Before this commit: robot ma_robot, 7 links, 6 joints
Links:
- link base_link: mass 2.899175 -> 2.899172
- link rplidar_s2_link: geometry collision mesh filename=package://ma_robot_description/meshes/ma_robot/rplidar_s2_l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 scale=0.01 0.01 0.01; visual mesh filename=package://ma_robot_description/meshes/ma_robot/rplidar_s2_l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 scale=1 1 1
- link zed2_camera_link: geometry collision mesh filename=package://ma_robot_description/meshes/ma_robot/zed2_camera_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 scale=0.01 0.01 0.01; visual mesh filename=package://ma_robot_description/meshes/ma_robot/zed2_camera_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 scale=1 1 1
Joints:
- joint front_left_wheel_joint: origin xyz=0.130000 0.060000 0.020000 rpy=-1.570796 0.000000 0.000000 -> xyz=0.012900 0.124477 -0.043048 rpy=-1.570796 0.000000 0.000000
- joint front_right_wheel_joint: origin xyz=0.130000 -0.185000 0.020000 rpy=1.570796 0.000000 0.000000 -> xyz=0.012900 0.001523 0.083048 rpy=1.570796 0.000000 0.000000
- joint rear_left_wheel_joint: origin xyz=-0.020000 0.060000 0.020000 rpy=-1.570796 0.000000 0.000000 -> xyz=-0.052900 0.132477 0.083048 rpy=-1.570796 0.000000 0.000000
- joint rear_right_wheel_joint: origin xyz=-0.020000 -0.187000 0.020000 rpy=1.570796 0.000000 0.000000 -> xyz=-0.052900 0.003523 -0.043048 rpy=1.570796 0.000000 0.000000

File: ma_robot_description/urdf/ma_robot.urdf.xacro (robot description, xacro)
@@ -2,26 +2,24 @@
 <robot xmlns:xacro="http://www.ros.org/wiki/xacro" name="ma_robot">
   <!-- Materials (shared across all assemblies) -->
+  <material name="Acetal_Resin_Black">
+    <color rgba="0.098 0.098 0.098 1.0"/>
+  </material>
   <material name="PA_11_Nylon_HP_11_30_with_EOS_P_396_3D_Printer">
     <color rgba="0.247 0.247 0.247 1.0"/>
   </material>
   <material name="Steel">
-    <color rgba="1.000 1.000 1.000 1.0"/>
-  </material>
-  <material name="Acetal_Resin_Black">
-    <color rgba="0.098 0.098 0.098 1.0"/>
+    <color rgba="0.627 0.627 0.627 1.0"/>
   </material>
   <!-- Assembly includes -->
+  <xacro:include filename="$(find ma_robot_description)/urdf/assemblies/rear_left_wheel_link.urdf.xacro"/>
   <xacro:include filename="$(find ma_robot_description)/urdf/assemblies/front_left_wheel_link.urdf.xacro"/>
   <xacro:include filename="$(find ma_robot_description)/urdf/assemblies/front_right_wheel_link.urdf.xacro"/>
-  <xacro:include filename="$(find ma_robot_description)/urdf/assemblies/rear_left_wheel_link.urdf.xacro"/>
   <xacro:include filename="$(find ma_robot_description)/urdf/assemblies/rear_right_wheel_link.urdf.xacro"/>
-  <xacro:include filename="$(find ma_robot_description)/urdf/assemblies/base_link.urdf.xacro"/>
   <xacro:include filename="$(find ma_robot_description)/urdf/assemblies/ma_robot.urdf.xacro"/>
   <!-- Instantiate assemblies -->
+  <xacro:rear_left_wheel_link prefix=""/>
   <xacro:front_left_wheel_link prefix=""/>
   <xacro:front_right_wheel_link prefix=""/>
-  <xacro:rear_left_wheel_link prefix=""/>
   <xacro:rear_right_wheel_link prefix=""/>
-  <xacro:base_link prefix=""/>
   <xacro:ma_robot prefix=""/>
   <!-- Mount joints (cross-assembly connections) -->
@@ -30,18 +28,15 @@
   <!-- update the include + macro call above, and adjust -->
   <!-- parent/child link names in the mount joint below. -->
-  <joint name="zed2_camera_joint" type="fixed">
+  <joint name="rear_left_wheel_joint" type="continuous">
     <parent link="base_link"/>
-    <child link="zed2_camera_link"/>
-    <origin xyz="0.145000 -0.062500 -0.007371" rpy="0.000000 0.000000 -1.570796"/>
-  </joint>
-  <joint name="rplidar_s2_joint" type="fixed">
-    <parent link="base_link"/>
-    <child link="rplidar_s2_link"/>
-    <origin xyz="-0.433747 -0.657506 0.046815" rpy="0.000000 0.000000 -1.570796"/>
+    <child link="rear_left_wheel_link"/>
+    <origin xyz="-0.052900 0.132477 0.083048" rpy="-1.570796 0.000000 0.000000"/>
+    <axis xyz="0.000000 0.000000 1.000000"/>
+    <limit effort="100.0" velocity="1.00"/>
   </joint>
   <joint name="front_right_wheel_joint" type="continuous">
     <parent link="base_link"/>
     <child link="front_right_wheel_link"/>
-    <origin xyz="0.130000 -0.185000 0.020000" rpy="1.570796 0.000000 0.000000"/>
+    <origin xyz="0.012900 0.001523 0.083048" rpy="1.570796 0.000000 0.000000"/>
     <axis xyz="0.000000 0.000000 1.000000"/>
     <limit effort="100.0" velocity="1.00"/>
@@ -50,5 +45,5 @@
     <parent link="base_link"/>
     <child link="rear_right_wheel_link"/>
-    <origin xyz="-0.020000 -0.187000 0.020000" rpy="1.570796 0.000000 0.000000"/>
+    <origin xyz="-0.052900 0.003523 -0.043048" rpy="1.570796 0.000000 0.000000"/>
     <axis xyz="0.000000 0.000000 1.000000"/>
     <limit effort="100.0" velocity="1.00"/>
@@ -57,12 +52,5 @@
     <parent link="base_link"/>
     <child link="front_left_wheel_link"/>
-    <origin xyz="0.130000 0.060000 0.020000" rpy="-1.570796 0.000000 0.000000"/>
-    <axis xyz="0.000000 0.000000 1.000000"/>
-    <limit effort="100.0" velocity="1.00"/>
-  </joint>
-  <joint name="rear_left_wheel_joint" type="continuous">
-    <parent link="base_link"/>
-    <child link="rear_left_wheel_link"/>
-    <origin xyz="-0.020000 0.060000 0.020000" rpy="-1.570796 0.000000 0.000000"/>
+    <origin xyz="0.012900 0.124477 -0.043048" rpy="-1.570796 0.000000 0.000000"/>
     <axis xyz="0.000000 0.000000 1.000000"/>
     <limit effort="100.0" velocity="1.00"/>
