Commit message: edit ma  pkg

File: ma_robot_description/urdf/assemblies/ma_robot.urdf.xacro (robot description, xacro)
@@ -1,24 +1,17 @@
 <?xml version="1.0"?>
-<robot xmlns:xacro="http://www.ros.org/wiki/xacro" name="base_link_macro">
-  <xacro:macro name="base_link" params="prefix">
+<robot xmlns:xacro="http://www.ros.org/wiki/xacro" name="ma_robot_macro">
+  <xacro:macro name="ma_robot" params="prefix">
     <!-- Links -->
     <link name="${prefix}base_link">
       <inertial>
-        <origin xyz="0.041588 -0.062494 0.024412" rpy="0 0 0"/>
-        <mass value="2.898778"/>
-        <inertia ixx="7.972007e-03" ixy="9.038509e-07" ixz="2.755930e-04"
-                 iyy="1.378869e-02" iyz="-4.482345e-07" izz="2.052341e-02"/>
+        <origin xyz="0.041574 -0.062494 0.024420" rpy="0 0 0"/>
+        <mass value="2.899152"/>
+        <inertia ixx="7.973742e-03" ixy="9.036729e-07" ixz="2.781740e-04"
+                 iyy="1.379462e-02" iyz="-4.481306e-07" izz="2.052761e-02"/>
       </inertial>
-      <visual>
-        <origin xyz="0.000000 0.000000 0.000000" rpy="0.000000 0.000000 0.000000"/>
-        <geometry>
-          <mesh filename="package://ma_robot_description/meshes/base_link/base_link.dae" scale="1 1 1"/>
-        </geometry>
-        <material name="Acetal_Resin_Black"/>
-      </visual>
       <collision>
         <origin xyz="0.000000 0.000000 0.000000" rpy="0.000000 0.000000 0.000000"/>
         <geometry>
-          <mesh filename="package://ma_robot_description/meshes/base_link/base_link_collision.stl" scale="0.01 0.01 0.01"/>
+          <mesh filename="package://ma_robot_description/meshes/ma_robot/base_link_collision.stl" scale="0.01 0.01 0.01"/>
         </geometry>
       </collision>
@@ -34,5 +27,5 @@
         <origin xyz="0.000000 0.000000 0.000000" rpy="0.000000 0.000000 0.000000"/>
         <geometry>
-          <mesh filename="package://ma_robot_description/meshes/base_link/zed2_camera_link.dae" scale="1 1 1"/>
+          <mesh filename="package://ma_robot_description/meshes/ma_robot/zed2_camera_link.dae" scale="1 1 1"/>
         </geometry>
         <material name="PA_11_Nylon_HP_11_30_with_EOS_P_396_3D_Printer"/>
@@ -41,5 +34,5 @@
         <origin xyz="0.000000 0.000000 0.000000" rpy="0.000000 0.000000 0.000000"/>
         <geometry>
-          <mesh filename="package://ma_robot_description/meshes/base_link/zed2_camera_link_collision.stl" scale="0.01 0.01 0.01"/>
+          <mesh filename="package://ma_robot_description/meshes/ma_robot/zed2_camera_link_collision.stl" scale="0.01 0.01 0.01"/>
         </geometry>
       </collision>
@@ -55,5 +48,5 @@
         <origin xyz="0.000000 0.000000 0.000000" rpy="0.000000 0.000000 0.000000"/>
         <geometry>
-          <mesh filename="package://ma_robot_description/meshes/base_link/rplidar_s2_link.dae" scale="1 1 1"/>
+          <mesh filename="package://ma_robot_description/meshes/ma_robot/rplidar_s2_link.dae" scale="1 1 1"/>
         </geometry>
         <material name="Steel"/>
@@ -62,5 +55,5 @@
         <origin xyz="0.000000 0.000000 0.000000" rpy="0.000000 0.000000 0.000000"/>
         <geometry>
-          <mesh filename="package://ma_robot_description/meshes/base_link/rplidar_s2_link_collision.stl" scale="0.01 0.01 0.01"/>
+          <mesh filename="package://ma_robot_description/meshes/ma_robot/rplidar_s2_link_collision.stl" scale="0.01 0.01 0.01"/>
         </geometry>
       </collision>

Commit message: Add Gazebo sensors and fix ZED2 camera orientation

File: ma_robot_description/urdf/assemblies/ma_robot.urdf.xacro (robot description, xacro)
@@ -36,6 +36,12 @@
     <!-- ZED2 camera -->
     <link name="${prefix}zed2_camera_link">
+      <!--
+        Camera link frame points forward with base_link +X.
+        The inertia transform preserves the original physical inertia.
+      -->
       <inertial>
-        <origin xyz="0.000000 0.015505 0.042389" rpy="0 0 0"/>
+        <origin
+          xyz="0.015505 0.000000 0.042389"
+          rpy="0.000000 0.000000 -1.570796"/>
         <mass value="0.178229"/>
         <inertia
@@ -47,6 +53,9 @@
           izz="4.390806e-04"/>
       </inertial>
+      <!-- Keep the camera mesh in its original physical orientation -->
       <visual>
-        <origin xyz="0 0 0" rpy="0 0 0"/>
+        <origin
+          xyz="0 0 0"
+          rpy="0.000000 0.000000 -1.570796"/>
         <geometry>
           <mesh
@@ -56,6 +65,9 @@
         <material name="PA_11_Nylon_HP_11_30_with_EOS_P_396_3D_Printer"/>
       </visual>
+      <!-- Keep the collision mesh aligned with the visual mesh -->
       <collision>
-        <origin xyz="0 0 0" rpy="0 0 0"/>
+        <origin
+          xyz="0 0 0"
+          rpy="0.000000 0.000000 -1.570796"/>
         <geometry>
           <mesh
@@ -100,5 +112,9 @@
       </collision>
     </link>
-    <!-- Camera fixed joint -->
+    <!--
+      Camera frame points forward.
+      Its yaw is now zero, so camera +X is aligned with base_link +X.
+      The -90 degree visual rotation above keeps the camera model unchanged.
+    -->
     <joint name="${prefix}zed2_camera_joint" type="fixed">
       <parent link="${prefix}base_link"/>
@@ -106,7 +122,7 @@
       <origin
         xyz="0.145000 -0.062500 -0.007371"
-        rpy="0.000000 0.000000 -1.570796"/>
+        rpy="0.000000 0.000000 0.000000"/>
     </joint>
-    <!-- Lidar fixed joint: frame positioned at physical lidar center -->
+    <!-- Lidar fixed joint -->
     <joint name="${prefix}rplidar_s2_joint" type="fixed">
       <parent link="${prefix}base_link"/>

File: ma_robot_description/urdf/ma_robot.gazebo.xacro (robot description, xacro)
@@ -26,27 +26,96 @@
     <kd>10.0</kd>
   </gazebo>
-  <!-- Four-wheel differential drive -->
+  <!-- RPLIDAR S2 simulation -->
+  <gazebo reference="rplidar_s2_link">
+    <sensor name="rplidar_s2_sensor" type="gpu_lidar">
+      <pose>0 0 0 0 0 0</pose>
+      <topic>/scan</topic>
+      <gz_frame_id>rplidar_s2_link</gz_frame_id>
+      <update_rate>10</update_rate>
+      <always_on>true</always_on>
+      <visualize>true</visualize>
+      <lidar>
+        <scan>
+          <horizontal>
+            <samples>720</samples>
+            <resolution>1</resolution>
+            <min_angle>-3.141592</min_angle>
+            <max_angle>3.141592</max_angle>
+          </horizontal>
+        </scan>
+        <range>
+          <min>0.15</min>
+          <max>30.0</max>
+          <resolution>0.01</resolution>
+        </range>
+        <noise>
+          <type>gaussian</type>
+          <mean>0.0</mean>
+          <stddev>0.01</stddev>
+        </noise>
+      </lidar>
+    </sensor>
+  </gazebo>
+  <!-- ZED2 RGB-D camera simulation -->
+  <gazebo reference="zed2_camera_link">
+    <sensor name="zed2_rgbd_sensor" type="rgbd_camera">
+      <!--
+        Sensor pose is zero because zed2_camera_link
+        now points forward with base_link +X.
+      -->
+      <pose>0 0 0 0 0 0</pose>
+      <topic>/camera</topic>
+      <gz_frame_id>zed2_camera_link</gz_frame_id>
+      <update_rate>30</update_rate>
+      <always_on>true</always_on>
+      <visualize>true</visualize>
+      <camera name="zed2_camera">
+        <horizontal_fov>1.92</horizontal_fov>
+        <image>
+          <width>640</width>
+          <height>480</height>
+          <format>R8G8B8</format>
+        </image>
+        <clip>
+          <near>0.10</near>
+          <far>20.0</far>
+        </clip>
+        <depth_camera>
+          <clip>
+            <near>0.20</near>
+            <far>20.0</far>
+          </clip>
+        </depth_camera>
+      </camera>
+    </sensor>
+  </gazebo>
+  <!-- Gazebo model systems -->
   <gazebo>
+    <!-- Publish wheel joint states -->
+    <plugin
+      filename="gz-sim-joint-state-publisher-system"
+      name="gz::sim::systems::JointStatePublisher">
+      <topic>joint_states</topic>
+      <joint_name>front_left_wheel_joint</joint_name>
+      <joint_name>front_right_wheel_joint</joint_name>
+      <joint_name>rear_left_wheel_joint</joint_name>
+      <joint_name>rear_right_wheel_joint</joint_name>
+    </plugin>
+    <!-- Four-wheel differential drive -->
     <plugin
       filename="gz-sim-diff-drive-system"
       name="gz::sim::systems::DiffDrive">
-      <!-- Left wheels -->
       <left_joint>front_left_wheel_joint</left_joint>
       <left_joint>rear_left_wheel_joint</left_joint>
-      <!-- Right wheels -->
       <right_joint>front_right_wheel_joint</right_joint>
       <right_joint>rear_right_wheel_joint</right_joint>
-      <!-- Robot dimensions -->
       <wheel_separation>0.246</wheel_separation>
       <wheel_radius>0.045</wheel_radius>
-      <!-- Gazebo topics -->
       <topic>cmd_vel</topic>
       <odom_topic>odom</odom_topic>
       <tf_topic>tf</tf_topic>
-      <!-- TF frames -->
       <frame_id>odom</frame_id>
       <child_frame_id>base_link</child_frame_id>
       <odom_publish_frequency>50</odom_publish_frequency>
-      <!-- Motion limits -->
       <max_linear_acceleration>1.0</max_linear_acceleration>
       <max_angular_acceleration>2.0</max_angular_acceleration>

Commit message: Improve Gazebo bridge, camera frames, and odometry

File: ma_robot_description/urdf/assemblies/ma_robot.urdf.xacro (robot description, xacro)
@@ -3,8 +3,11 @@
        name="ma_robot_macro">
   <xacro:macro name="ma_robot" params="prefix">
+    <link name="${prefix}base_footprint"/>
     <!-- Base link -->
     <link name="${prefix}base_link">
       <inertial>
-        <origin xyz="0.041574 -0.062494 0.024420" rpy="0 0 0"/>
+        <origin
+          xyz="0.041574 -0.062494 0.024420"
+          rpy="0 0 0"/>
         <mass value="2.899172"/>
         <inertia
@@ -34,9 +37,26 @@
       </collision>
     </link>
-    <!-- ZED2 camera -->
+    <!--
+      The base_link CAD origin is offset from the kinematic
+      center represented by base_footprint.
+      X = -55.000 mm
+      Y = +62.500 mm
+      Z = +26.386 mm above the ground
+    -->
+    <joint name="${prefix}base_footprint_joint"
+           type="fixed">
+      <parent link="${prefix}base_footprint"/>
+      <child link="${prefix}base_link"/>
+      <origin
+        xyz="-0.055000 0.062500 0.026386"
+        rpy="0.000000 0.000000 0.000000"/>
+    </joint>
+    <!-- ZED2 camera physical link -->
     <link name="${prefix}zed2_camera_link">
       <!--
-        Camera link frame points forward with base_link +X.
-        The inertia transform preserves the original physical inertia.
+        zed2_camera_link uses the standard robot frame:
+          +X forward
+          +Y left
+          +Z upward
       -->
       <inertial>
@@ -53,5 +73,4 @@
           izz="4.390806e-04"/>
       </inertial>
-      <!-- Keep the camera mesh in its original physical orientation -->
       <visual>
         <origin
@@ -63,7 +82,7 @@
             scale="1 1 1"/>
         </geometry>
-        <material name="PA_11_Nylon_HP_11_30_with_EOS_P_396_3D_Printer"/>
+        <material
+          name="PA_11_Nylon_HP_11_30_with_EOS_P_396_3D_Printer"/>
       </visual>
-      <!-- Keep the collision mesh aligned with the visual mesh -->
       <collision>
         <origin
@@ -77,4 +96,14 @@
       </collision>
     </link>
+    <!--
+      ZED2 optical frame.
+      ROS optical frame convention:
+        +Z points forward through the camera lens
+        +X points to the right in the image
+        +Y points downward in the image
+      This is a virtual reference frame, therefore it does not
+      require visual, collision, mass, or inertia properties.
+    -->
+    <link name="${prefix}zed2_camera_optical_link"/>
     <!-- RPLIDAR S2 -->
     <link name="${prefix}rplidar_s2_link">
@@ -92,5 +121,5 @@
           izz="2.370283e-04"/>
       </inertial>
-      <!-- Offset removes the coordinates baked inside the DAE mesh -->
+      <!-- Offset removes coordinates baked inside the DAE mesh -->
       <visual>
         <origin
@@ -108,14 +137,13 @@
         <origin xyz="0 0 0" rpy="0 0 0"/>
         <geometry>
-          <cylinder radius="0.0385" length="0.038851"/>
+          <cylinder
+            radius="0.0385"
+            length="0.038851"/>
         </geometry>
       </collision>
     </link>
-    <!--
-      Camera frame points forward.
-      Its yaw is now zero, so camera +X is aligned with base_link +X.
-      The -90 degree visual rotation above keeps the camera model unchanged.
-    -->
-    <joint name="${prefix}zed2_camera_joint" type="fixed">
+    <!-- Camera fixed joint -->
+    <joint name="${prefix}zed2_camera_joint"
+           type="fixed">
       <parent link="${prefix}base_link"/>
       <child link="${prefix}zed2_camera_link"/>
@@ -124,6 +152,19 @@
         rpy="0.000000 0.000000 0.000000"/>
     </joint>
+    <!--
+      Fixed transform from the physical camera frame to the
+      standard ROS optical camera frame.
+    -->
+    <joint name="${prefix}zed2_camera_optical_joint"
+           type="fixed">
+      <parent link="${prefix}zed2_camera_link"/>
+      <child link="${prefix}zed2_camera_optical_link"/>
+      <origin
+        xyz="0.000000 0.000000 0.000000"
+        rpy="-1.570796 0.000000 -1.570796"/>
+    </joint>
     <!-- Lidar fixed joint -->
-    <joint name="${prefix}rplidar_s2_joint" type="fixed">
+    <joint name="${prefix}rplidar_s2_joint"
+           type="fixed">
       <parent link="${prefix}base_link"/>
       <child link="${prefix}rplidar_s2_link"/>

File: ma_robot_description/urdf/ma_robot.gazebo.xacro (robot description, xacro)
@@ -62,5 +62,5 @@
       <!--
         Sensor pose is zero because zed2_camera_link
-        now points forward with base_link +X.
+        points forward with base_link +X.
       -->
       <pose>0 0 0 0 0 0</pose>
@@ -106,15 +106,24 @@
       filename="gz-sim-diff-drive-system"
       name="gz::sim::systems::DiffDrive">
+      <!-- Left wheels -->
       <left_joint>front_left_wheel_joint</left_joint>
       <left_joint>rear_left_wheel_joint</left_joint>
+      <!-- Right wheels -->
       <right_joint>front_right_wheel_joint</right_joint>
       <right_joint>rear_right_wheel_joint</right_joint>
+      <!-- Robot dimensions -->
       <wheel_separation>0.246</wheel_separation>
       <wheel_radius>0.045</wheel_radius>
+      <!-- Command and odometry topics -->
       <topic>cmd_vel</topic>
       <odom_topic>odom</odom_topic>
       <tf_topic>tf</tf_topic>
+      <!--
+        Gazebo publishes odom -> base_footprint.
+        robot_state_publisher publishes
+        base_footprint -> base_link.
+      -->
       <frame_id>odom</frame_id>
-      <child_frame_id>base_link</child_frame_id>
+      <child_frame_id>base_footprint</child_frame_id>
       <odom_publish_frequency>50</odom_publish_frequency>
       <max_linear_acceleration>1.0</max_linear_acceleration>
