Commit message: Add Gazebo simulation and fix robot wheel configuration

File: ma_robot_description/urdf/ma_robot.urdf.xacro (robot description, xacro)
@@ -1,5 +1,5 @@
 <?xml version="1.0"?>
 <robot xmlns:xacro="http://www.ros.org/wiki/xacro" name="ma_robot">
-  <!-- Materials (shared across all assemblies) -->
+  <!-- Materials -->
   <material name="Acetal_Resin_Black">
     <color rgba="0.098 0.098 0.098 1.0"/>
@@ -17,4 +17,6 @@
   <xacro:include filename="$(find ma_robot_description)/urdf/assemblies/rear_right_wheel_link.urdf.xacro"/>
   <xacro:include filename="$(find ma_robot_description)/urdf/assemblies/ma_robot.urdf.xacro"/>
+  <!-- Gazebo configuration -->
+  <xacro:include filename="$(find ma_robot_description)/urdf/ma_robot.gazebo.xacro"/>
   <!-- Instantiate assemblies -->
   <xacro:rear_left_wheel_link prefix=""/>
@@ -32,5 +34,5 @@
       rpy="-1.570796 0.000000 0.000000"/>
     <axis xyz="0.000000 0.000000 1.000000"/>
-    <limit effort="100.0" velocity="1.00"/>
+    <limit effort="100.0" velocity="10.0"/>
   </joint>
   <!-- Front-right wheel -->
@@ -41,6 +43,7 @@
       xyz="0.130000 -0.185000 0.020000"
       rpy="1.570796 0.000000 0.000000"/>
-    <axis xyz="0.000000 0.000000 1.000000"/>
-    <limit effort="100.0" velocity="1.00"/>
+    <!-- Reversed because the right wheel frame is mirrored -->
+    <axis xyz="0.000000 0.000000 -1.000000"/>
+    <limit effort="100.0" velocity="10.0"/>
   </joint>
   <!-- Rear-left wheel -->
@@ -52,5 +55,5 @@
       rpy="-1.570796 0.000000 0.000000"/>
     <axis xyz="0.000000 0.000000 1.000000"/>
-    <limit effort="100.0" velocity="1.00"/>
+    <limit effort="100.0" velocity="10.0"/>
   </joint>
   <!-- Rear-right wheel -->
@@ -61,8 +64,9 @@
       xyz="-0.020000 -0.187000 0.020000"
       rpy="1.570796 0.000000 0.000000"/>
-    <axis xyz="0.000000 0.000000 1.000000"/>
-    <limit effort="100.0" velocity="1.00"/>
+    <!-- Reversed because the right wheel frame is mirrored -->
+    <axis xyz="0.000000 0.000000 -1.000000"/>
+    <limit effort="100.0" velocity="10.0"/>
   </joint>
-  <!-- ROS 2 control: generated generic system -->
+  <!-- ROS 2 control -->
   <ros2_control name="ma_robot_system" type="system">
     <hardware>
