Commit message: Rename ma_robot_description → mabot_description; update package, CMake, URDF, xacro, launches, world, README, and metadata

File: mabot_description/urdf/assemblies/front_left_wheel_link.urdf.xacro (robot description, xacro)
@@ -21,5 +21,5 @@
         <geometry>
           <mesh
-            filename="package://ma_robot_description/meshes/front_left_wheel_link/front_left_wheel_link.dae"
+            filename="package://mabot_description/meshes/front_left_wheel_link/front_left_wheel_link.dae"
             scale="1 1 1"/>
         </geometry>

File: mabot_description/urdf/assemblies/front_right_wheel_link.urdf.xacro (robot description, xacro)
@@ -21,5 +21,5 @@
         <geometry>
           <mesh
-            filename="package://ma_robot_description/meshes/front_right_wheel_link/front_right_wheel_link.dae"
+            filename="package://mabot_description/meshes/front_right_wheel_link/front_right_wheel_link.dae"
             scale="1 1 1"/>
         </geometry>

File: mabot_description/urdf/assemblies/mabot.urdf.xacro (robot description, xacro)
@@ -1,6 +1,6 @@
 <?xml version="1.0"?>
 <robot xmlns:xacro="http://www.ros.org/wiki/xacro"
-       name="ma_robot_macro">
-  <xacro:macro name="ma_robot" params="prefix">
+    name="mabot_macro">
+  <xacro:macro name="mabot" params="prefix">
     <link name="${prefix}base_footprint"/>
     <!-- Base link -->
@@ -23,5 +23,5 @@
         <geometry>
           <mesh
-            filename="package://ma_robot_description/meshes/ma_robot/base_link.dae"
+            filename="package://mabot_description/meshes/ma_robot/base_link.dae"
             scale="1 1 1"/>
         </geometry>
@@ -32,5 +32,5 @@
         <geometry>
           <mesh
-            filename="package://ma_robot_description/meshes/ma_robot/base_link_collision.stl"
+            filename="package://mabot_description/meshes/ma_robot/base_link_collision.stl"
             scale="0.01 0.01 0.01"/>
         </geometry>
@@ -79,5 +79,5 @@
         <geometry>
           <mesh
-            filename="package://ma_robot_description/meshes/ma_robot/zed2_camera_link.dae"
+            filename="package://mabot_description/meshes/ma_robot/zed2_camera_link.dae"
             scale="1 1 1"/>
         </geometry>
@@ -91,5 +91,5 @@
         <geometry>
           <mesh
-            filename="package://ma_robot_description/meshes/ma_robot/zed2_camera_link_collision.stl"
+            filename="package://mabot_description/meshes/ma_robot/zed2_camera_link_collision.stl"
             scale="0.01 0.01 0.01"/>
         </geometry>
@@ -128,5 +128,5 @@
         <geometry>
           <mesh
-            filename="package://ma_robot_description/meshes/ma_robot/rplidar_s2_link.dae"
+            filename="package://mabot_description/meshes/ma_robot/rplidar_s2_link.dae"
             scale="1 1 1"/>
         </geometry>

File: mabot_description/urdf/assemblies/rear_left_wheel_link.urdf.xacro (robot description, xacro)
@@ -1,7 +1,7 @@
 <?xml version="1.0"?>
 <robot xmlns:xacro="http://www.ros.org/wiki/xacro"
-       name="rear_right_wheel_link_macro">
-  <xacro:macro name="rear_right_wheel_link" params="prefix">
-    <link name="${prefix}rear_right_wheel_link">
+       name="rear_left_wheel_link_macro">
+  <xacro:macro name="rear_left_wheel_link" params="prefix">
+    <link name="${prefix}rear_left_wheel_link">
       <inertial>
         <origin xyz="0 0 0" rpy="0 0 0"/>
@@ -17,9 +17,9 @@
       <visual>
         <origin
-          xyz="0.002378 -0.018051 -0.241816"
+          xyz="-0.012900 -0.018051 0.005477"
           rpy="1.570796 0.000000 0.000000"/>
         <geometry>
           <mesh
-            filename="package://ma_robot_description/meshes/rear_right_wheel_link/rear_right_wheel_link.dae"
+            filename="package://mabot_description/meshes/rear_left_wheel_link/rear_left_wheel_link.dae"
             scale="1 1 1"/>
         </geometry>

File: mabot_description/urdf/assemblies/rear_right_wheel_link.urdf.xacro (robot description, xacro)
@@ -1,7 +1,7 @@
 <?xml version="1.0"?>
 <robot xmlns:xacro="http://www.ros.org/wiki/xacro"
-       name="rear_left_wheel_link_macro">
-  <xacro:macro name="rear_left_wheel_link" params="prefix">
-    <link name="${prefix}rear_left_wheel_link">
+       name="rear_right_wheel_link_macro">
+  <xacro:macro name="rear_right_wheel_link" params="prefix">
+    <link name="${prefix}rear_right_wheel_link">
       <inertial>
         <origin xyz="0 0 0" rpy="0 0 0"/>
@@ -17,9 +17,9 @@
       <visual>
         <origin
-          xyz="-0.012900 -0.018051 0.005477"
+          xyz="0.002378 -0.018051 -0.241816"
           rpy="1.570796 0.000000 0.000000"/>
         <geometry>
           <mesh
-            filename="package://ma_robot_description/meshes/rear_left_wheel_link/rear_left_wheel_link.dae"
+            filename="package://mabot_description/meshes/rear_right_wheel_link/rear_right_wheel_link.dae"
             scale="1 1 1"/>
         </geometry>

File: mabot_description/urdf/mabot.urdf (robot description, URDF)
Before this commit: robot ma_robot, 7 links, 6 joints
Links:
- link base_link: geometry collision mesh filename=package://mabot_description/meshes/ma_robot/base_link_colli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 scale=0.01 0.01 0.01; visual mesh filename=package://mabot_description/meshes/ma_robot/base_link.dae scale=1 1 1
- link front_left_wheel_link: geometry collision cylinder length=0.050 radius=0.045; visual mesh filename=package://mabot_description/meshes/front_left_wheel_link/fr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 scale=1 1 1
- link front_right_wheel_link: geometry collision cylinder length=0.050 radius=0.045; visual mesh filename=package://mabot_description/meshes/front_right_wheel_link/f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 scale=1 1 1
- link rear_left_wheel_link: geometry collision cylinder length=0.050 radius=0.045; visual mesh filename=package://mabot_description/meshes/rear_left_wheel_link/rea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 scale=1 1 1
- link rear_right_wheel_link: geometry collision cylinder length=0.050 radius=0.045; visual mesh filename=package://mabot_description/meshes/rear_right_wheel_link/re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 scale=1 1 1
- link rplidar_s2_link: geometry collision mesh filename=package://mabot_description/meshes/ma_robot/rplidar_s2_link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 scale=0.01 0.01 0.01; visual mesh filename=package://mabot_description/meshes/ma_robot/rplidar_s2_link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 scale=1 1 1
- link zed2_camera_link: geometry collision mesh filename=package://mabot_description/meshes/ma_robot/zed2_camera_lin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 scale=0.01 0.01 0.01; visual mesh filename=package://mabot_description/meshes/ma_robot/zed2_camera_lin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 scale=1 1 1

File: mabot_description/urdf/mabot.urdf.xacro (robot description, xacro)
@@ -1,4 +1,4 @@
 <?xml version="1.0"?>
-<robot xmlns:xacro="http://www.ros.org/wiki/xacro" name="ma_robot">
+<robot xmlns:xacro="http://www.ros.org/wiki/xacro" name="mabot">
   <!-- Materials -->
   <material name="Acetal_Resin_Black">
@@ -12,11 +12,11 @@
   </material>
   <!-- Assembly includes -->
-  <xacro:include filename="$(find ma_robot_description)/urdf/assemblies/rear_left_wheel_link.urdf.xacro"/>
-  <xacro:include filename="$(find ma_robot_description)/urdf/assemblies/front_left_wheel_link.urdf.xacro"/>
-  <xacro:include filename="$(find ma_robot_description)/urdf/assemblies/front_right_wheel_link.urdf.xacro"/>
-  <xacro:include filename="$(find ma_robot_description)/urdf/assemblies/rear_right_wheel_link.urdf.xacro"/>
-  <xacro:include filename="$(find ma_robot_description)/urdf/assemblies/ma_robot.urdf.xacro"/>
+  <xacro:include filename="$(find mabot_description)/urdf/assemblies/rear_left_wheel_link.urdf.xacro"/>
+  <xacro:include filename="$(find mabot_description)/urdf/assemblies/front_left_wheel_link.urdf.xacro"/>
+  <xacro:include filename="$(find mabot_description)/urdf/assemblies/front_right_wheel_link.urdf.xacro"/>
+  <xacro:include filename="$(find mabot_description)/urdf/assemblies/rear_right_wheel_link.urdf.xacro"/>
+  <xacro:include filename="$(find mabot_description)/urdf/assemblies/mabot.urdf.xacro"/>
   <!-- Gazebo configuration -->
-  <xacro:include filename="$(find ma_robot_description)/urdf/ma_robot.gazebo.xacro"/>
+  <xacro:include filename="$(find mabot_description)/urdf/mabot.gazebo.xacro"/>
   <!-- Instantiate assemblies -->
   <xacro:rear_left_wheel_link prefix=""/>
@@ -24,5 +24,5 @@
   <xacro:front_right_wheel_link prefix=""/>
   <xacro:rear_right_wheel_link prefix=""/>
-  <xacro:ma_robot prefix=""/>
+  <xacro:mabot prefix=""/>
   <!-- Wheel mount joints -->
   <!-- Front-left wheel -->
@@ -69,9 +69,9 @@
   </joint>
   <!-- ROS 2 control -->
-  <ros2_control name="ma_robot_system" type="system">
+  <ros2_control name="mabot_system" type="system">
     <hardware>
       <plugin>mock_components/GenericSystem</plugin>
-      <param name="cmd_topic">sim/ma_robot_system/cmd</param>
-      <param name="state_topic">sim/ma_robot_system/state</param>
+      <param name="cmd_topic">sim/mabot_system/cmd</param>
+      <param name="state_topic">sim/mabot_system/state</param>
     </hardware>
     <joint name="front_left_wheel_joint">
