Commit message: update pkg

File: mabot_description/urdf/assemblies/mabot.urdf.xacro (robot description, xacro)
@@ -1,13 +1,24 @@
 <?xml version="1.0"?>
 <robot xmlns:xacro="http://www.ros.org/wiki/xacro"
-    name="mabot_macro">
+       name="mabot_macro">
   <xacro:macro name="mabot" params="prefix">
+    <!-- ================================================== -->
+    <!-- Base footprint                                     -->
+    <!-- ================================================== -->
+    <!--
+      Virtual ground-level frame used as the robot's
+      kinematic reference.
+      It intentionally has no visual, collision, mass,
+      or inertia properties.
+    -->
     <link name="${prefix}base_footprint"/>
-    <!-- Base link -->
+    <!-- ================================================== -->
+    <!-- Base link                                          -->
+    <!-- ================================================== -->
     <link name="${prefix}base_link">
       <inertial>
         <origin
           xyz="0.041574 -0.062494 0.024420"
-          rpy="0 0 0"/>
+          rpy="0.000000 0.000000 0.000000"/>
         <mass value="2.899172"/>
         <inertia
@@ -20,5 +31,7 @@
       </inertial>
       <visual>
-        <origin xyz="0 0 0" rpy="0 0 0"/>
+        <origin
+          xyz="0.000000 0.000000 0.000000"
+          rpy="0.000000 0.000000 0.000000"/>
         <geometry>
           <mesh
@@ -29,5 +42,7 @@
       </visual>
       <collision>
-        <origin xyz="0 0 0" rpy="0 0 0"/>
+        <origin
+          xyz="0.000000 0.000000 0.000000"
+          rpy="0.000000 0.000000 0.000000"/>
         <geometry>
           <mesh
@@ -52,5 +67,7 @@
         rpy="0.000000 0.000000 0.000000"/>
     </joint>
-    <!-- ZED2 camera physical link -->
+    <!-- ================================================== -->
+    <!-- ZED2 camera physical link                          -->
+    <!-- ================================================== -->
     <link name="${prefix}zed2_camera_link">
       <!--
@@ -59,4 +76,6 @@
           +Y left
           +Z upward
+        The inertia transform preserves the original
+        physical inertia exported from Fusion 360.
       -->
       <inertial>
@@ -73,7 +92,11 @@
           izz="4.390806e-04"/>
       </inertial>
+      <!--
+        Keep the camera mesh in its original physical
+        mounting orientation.
+      -->
       <visual>
         <origin
-          xyz="0 0 0"
+          xyz="0.000000 0.000000 0.000000"
           rpy="0.000000 0.000000 -1.570796"/>
         <geometry>
@@ -85,7 +108,11 @@
           name="PA_11_Nylon_HP_11_30_with_EOS_P_396_3D_Printer"/>
       </visual>
+      <!--
+        Keep the collision mesh aligned with the
+        visible camera mesh.
+      -->
       <collision>
         <origin
-          xyz="0 0 0"
+          xyz="0.000000 0.000000 0.000000"
           rpy="0.000000 0.000000 -1.570796"/>
         <geometry>
@@ -96,20 +123,33 @@
       </collision>
     </link>
-    <!--
-      ZED2 optical frame.
-      ROS optical frame convention:
+    <!-- ================================================== -->
+    <!-- ZED2 optical frame                                 -->
+    <!-- ================================================== -->
+    <!--
+      ROS optical-frame convention:
         +Z points forward through the camera lens
         +X points to the right in the image
         +Y points downward in the image
-      This is a virtual reference frame, therefore it does not
-      require visual, collision, mass, or inertia properties.
+      This is a virtual reference frame and therefore does
+      not require visual, collision, mass or inertia.
     -->
     <link name="${prefix}zed2_camera_optical_link"/>
-    <!-- RPLIDAR S2 -->
+    <!-- ================================================== -->
+    <!-- RPLIDAR S2                                         -->
+    <!-- ================================================== -->
     <link name="${prefix}rplidar_s2_link">
+      <!--
+        The LiDAR link frame is aligned with base_link:
+          +X forward
+          +Y left
+          +Z upward
+        The inertial pose was transformed from the original
+        Fusion frame so that the physical inertia remains
+        unchanged after correcting the link orientation.
+      -->
       <inertial>
         <origin
-          xyz="-0.000007 -0.000076 -0.009381"
-          rpy="0 0 0"/>
+          xyz="-0.000076 0.000007 -0.009381"
+          rpy="0.000000 0.000000 -1.570796"/>
         <mass value="0.203764"/>
         <inertia
@@ -121,9 +161,15 @@
           izz="2.370283e-04"/>
       </inertial>
-      <!-- Offset removes coordinates baked inside the DAE mesh -->
+      <!--
+        The COLLADA mesh contains coordinates baked relative
+        to the original Fusion 360 assembly.
+        This transformed translation and rotation preserve
+        the original visible position while allowing the
+        rplidar_s2_link frame to point forward.
+      -->
       <visual>
         <origin
-          xyz="0.595006 -0.533018 -0.022261"
-          rpy="0 0 0"/>
+          xyz="-0.533018 -0.595006 -0.022261"
+          rpy="0.000000 0.000000 -1.570796"/>
         <geometry>
           <mesh
@@ -133,7 +179,14 @@
         <material name="Steel"/>
       </visual>
-      <!-- Simplified collision centered on the lidar frame -->
+      <!--
+        Simplified cylindrical collision centered on the
+        physical LiDAR frame.
+        A yaw rotation is unnecessary because the cylinder
+        is symmetric around its Z axis.
+      -->
       <collision>
-        <origin xyz="0 0 0" rpy="0 0 0"/>
+        <origin
+          xyz="0.000000 0.000000 0.000000"
+          rpy="0.000000 0.000000 0.000000"/>
         <geometry>
           <cylinder
@@ -143,5 +196,11 @@
       </collision>
     </link>
-    <!-- Camera fixed joint -->
+    <!-- ================================================== -->
+    <!-- Camera joints                                      -->
+    <!-- ================================================== -->
+    <!--
+      Camera physical frame aligned with the robot's
+      forward +X direction.
+    -->
     <joint name="${prefix}zed2_camera_joint"
            type="fixed">
@@ -164,5 +223,16 @@
         rpy="-1.570796 0.000000 -1.570796"/>
     </joint>
-    <!-- Lidar fixed joint -->
+    <!-- ================================================== -->
+    <!-- LiDAR joint                                        -->
+    <!-- ================================================== -->
+    <!--
+      The LiDAR frame is located at the physical sensor
+      center and aligned with the robot:
+        +X forward
+        +Y left
+        +Z upward
+      This alignment allows LaserScan angle 0 to represent
+      the front of MABot correctly.
+    -->
     <joint name="${prefix}rplidar_s2_joint"
            type="fixed">
@@ -171,5 +241,5 @@
       <origin
         xyz="0.099271 -0.062500 0.069076"
-        rpy="0.000000 0.000000 -1.570796"/>
+        rpy="0.000000 0.000000 0.000000"/>
     </joint>
   </xacro:macro>
